File: pcb/thingy.sch (KiCad schematic (older format))
At the start: 1 part

Commit message: new symbols and footprint library stub
Parts:
- removed U?: 7402, symbol 74xx:7402
- added U1: 2x18650_holder, thingy:2x18650_holder, symbol thingy:2x18650_holder
Changed lines of the file:
@@
 EESchema Schematic File Version 4
+LIBS:thingy-cache
 EELAYER 26 0
 EELAYER END
@@
 $EndDescr
 $Comp
-L 74xx:7402 U?
-U 1 1 5B93AAD5
-P 5500 3450
-F 0 "U?" H 5500 3775 50  0000 C CNN
-F 1 "7402" H 5500 3684 50  0000 C CNN
-F 2 "" H 5500 3450 50  0001 C CNN
-F 3 "http://www.ti.com/lit/gpn/sn7402" H 5500 3450 50  0001 C CNN
-	1    5500 3450
+L thingy:2x18650_holder U1
+U 1 1 5B93B1E9
+P 4750 3500
+F 0 "U1" H 4750 3825 50  0000 C CNN
+F 1 "2x18650_holder" H 4750 3734 50  0000 C CNN
+F 2 "thingy:2x18650_holder" V 4750 3500 50  0001 C CNN
+F 3 "" V 4750 3500 50  0001 C CNN
+	1    4750 3500
 	1    0    0    -1
 $EndComp

Commit message: few new elements & power module circuit
Parts:
- added C1, C2: 0.1u, symbol Device:C
- added C3: 10u, symbol Device:C
- added D1: G, symbol Device:LED
- added D2: R, symbol Device:LED
- added J1: USB_B_Micro, Connector_USB:USB_Micro-B_Molex-105017-0001, symbol Connector:USB_B_Micro
- added R1, R2, R4: 1k, symbol Device:R
- added R3: 1k2, symbol Device:R
- added R5: 100, symbol Device:R
- added U2: TP4056-B, symbol thingy:TP4056-B
- added U3: DW01A, symbol thingy:DW01A
- added U4: FS8205A, symbol thingy:FS8205A
- added U5: FT232RL, Package_SO:SSOP-28_5.3x10.2mm_P0.65mm, symbol Interface_USB:FT232RL
Connections:
- net labels added: +5V, BAT-, GND, VCC
- wire segments 0 -> 71
Other:
- note added: "powering module & battery\n"

Commit message: mss22d18 footprint added
Parts:
- added SW?: SW_DPDT_x2, symbol Switch:SW_DPDT_x2
- added U?: ESP-07, RF_Module:ESP-07, symbol RF_Module:ESP-07
Connections:
- wire segments 71 -> 74
Changed lines of the file:
@@
 Text Notes 5800 3050 0    79   ~ 0
 powering module & battery\n
+$Comp
+L Switch:SW_DPDT_x2 SW?
+U 1 1 5BABD89F
+P 3900 4250
+F 0 "SW?" H 3900 4535 50  0000 C CNN
+F 1 "SW_DPDT_x2" H 3900 4444 50  0000 C CNN
+F 2 "" H 3900 4250 50  0001 C CNN
+F 3 "" H 3900 4250 50  0001 C CNN
+	1    3900 4250
+	0    -1   -1   0
+$EndComp
+$Comp
+L RF_Module:ESP-07 U?
+U 1 1 5BAD4E4E
+P 3900 5500
+F 0 "U?" H 3900 6478 50  0000 C CNN
+F 1 "ESP-07" H 3900 6387 50  0000 C CNN
+F 2 "RF_Module:ESP-07" H 3900 5500 50  0001 C CNN
+F 3 "http://wiki.ai-thinker.com/_media/esp8266/esp8266_series_modules_user_manual_v1.1.pdf" H 3550 5600 50  0001 C CNN
+	1    3900 5500
+	1    0    0    -1
+$EndComp
+Wire Wire Line
+	3900 4450 3900 4700
+$Comp
+L power:VCC #PWR?
+U 1 1 5BAD9D59
+P 3800 3850
+F 0 "#PWR?" H 3800 3700 50  0001 C CNN
+F 1 "VCC" H 3817 4023 50  0000 C CNN
+F 2 "" H 3800 3850 50  0001 C CNN
+F 3 "" H 3800 3850 50  0001 C CNN
+	1    3800 3850
+	1    0    0    -1
+$EndComp
+Wire Wire Line
+	3800 3850 3800 4050
+$Comp
+L power:GND #PWR?
+U 1 1 5BADC7AF
+P 3900 6400
+F 0 "#PWR?" H 3900 6150 50  0001 C CNN
+F 1 "GND" H 3905 6227 50  0000 C CNN
+F 2 "" H 3900 6400 50  0001 C CNN
+F 3 "" H 3900 6400 50  0001 C CNN
+	1    3900 6400
+	1    0    0    -1
+$EndComp
+Wire Wire Line
+	3900 6200 3900 6400
 $EndSCHEMATC

Commit message: more schematic work
Parts:
- removed U5: FT232RL, Package_SO:SSOP-28_5.3x10.2mm_P0.65mm, symbol Interface_USB:FT232RL
- added J2: FLASH_JUMPER, Connector_PinHeader_2.54mm:PinHeader_1x02_P2.54mm_Vertical, symbol Connector:Conn_01x02_Male
- added J3: Conn_01x04_Male, Connector_PinHeader_2.54mm:PinHeader_1x04_P2.54mm_Vertical, symbol Connector:Conn_01x04_Male
- added R10, R11, R7, R9: 4k7, Resistor_SMD:R_1206_3216Metric, symbol Device:R
- added R12, R8: 1k, Resistor_SMD:R_1206_3216Metric, symbol Device:R
- added R6: R, Resistor_SMD:R_1206_3216Metric, symbol Device:R
- added SW2: SW_Push, symbol Switch:SW_Push
- C1: renamed from C2; footprint (none) -> Capacitor_SMD:C_1206_3216Metric
- C2: renamed from C3; footprint (none) -> Capacitor_SMD:C_1206_3216Metric
- C3: renamed from C1; footprint (none) -> Capacitor_SMD:C_1206_3216Metric
- D1, D2: footprint (none) -> LED_SMD:LED_1206_3216Metric
- R1: renamed from R5; footprint (none) -> Resistor_SMD:R_1206_3216Metric
- R2: renamed from R1; footprint (none) -> Resistor_SMD:R_1206_3216Metric
- R3: renamed from R2; footprint (none) -> Resistor_SMD:R_1206_3216Metric
- R4: footprint (none) -> Resistor_SMD:R_1206_3216Metric
- R5: renamed from R3; footprint (none) -> Resistor_SMD:R_1206_3216Metric
- U1: renamed from U3; footprint (none) -> Package_TO_SOT_SMD:SOT-23-6
- U2: footprint (none) -> Package_SO:SOIC-8_3.9x4.9mm_P1.27mm
- U4: footprint (none) -> Package_SO:TSSOP-8_4.4x3mm_P0.65mm
- gave numbers to parts that had none: 2
- renumbered U1 to U3
Connections:
- net labels added: I2C_SCL, I2C_SDA, RXD, TXD
- wire segments 74 -> 122

Commit message: dalsze prace
Parts:
- added J4: Conn_01x04_Male, Connector_PinHeader_2.54mm:PinHeader_1x04_P2.54mm_Vertical, symbol Connector:Conn_01x04_Male
- SW1: footprint (none) -> thingy:MSS22D18
Connections:
- wire segments 122 -> 126
Changed lines of the file:
@@
 F 0 "SW1" H 3900 4535 50  0000 C CNN
 F 1 "SW_DPDT_x2" H 3900 4444 50  0000 C CNN
-F 2 "" H 3900 4250 50  0001 C CNN
+F 2 "thingy:MSS22D18" H 3900 4250 50  0001 C CNN
 F 3 "" H 3900 4250 50  0001 C CNN
 	1    3900 4250
@@
 Wire Wire Line
 	6650 5250 6550 5250
+$Comp
+L Connector:Conn_01x04_Male J4
+U 1 1 5BB6A3AF
+P 6850 5900
+F 0 "J4" H 7100 5600 50  0000 R CNN
+F 1 "Conn_01x04_Male" H 7400 6100 50  0000 R CNN
+F 2 "Connector_PinHeader_2.54mm:PinHeader_1x04_P2.54mm_Vertical" H 6850 5900 50  0001 C CNN
+F 3 "~" H 6850 5900 50  0001 C CNN
+	1    6850 5900
+	-1   0    0    1
+$EndComp
+Text GLabel 6550 5700 0    50   Input ~ 0
+VCC
+Text GLabel 6550 5800 0    50   Input ~ 0
+GND
+Text GLabel 6550 5900 0    50   Input ~ 0
+I2C_SCL
+Text GLabel 6550 6000 0    50   Input ~ 0
+I2C_SDA
+Wire Wire Line
+	6550 5700 6650 5700
+Wire Wire Line
+	6650 5800 6550 5800
+Wire Wire Line
+	6550 5900 6650 5900
+Wire Wire Line
+	6650 6000 6550 6000
 $EndSCHEMATC

Commit message: thingy work in progress
Parts:
- J2: value FLASH_JUMPER -> FLASH
- J3: value Conn_01x04_Male -> PROG
- J4: value Conn_01x04_Male -> I2C
- SW1: value SW_DPDT_x2 -> POWER
- SW2: value SW_Push -> RESET; footprint (none) -> thingy:SUNROM_4388
Changed lines of the file:
@@
 P 3900 4250
 F 0 "SW1" H 3900 4535 50  0000 C CNN
-F 1 "SW_DPDT_x2" H 3900 4444 50  0000 C CNN
+F 1 "POWER" H 3900 4444 50  0000 C CNN
 F 2 "thingy:MSS22D18" H 3900 4250 50  0001 C CNN
 F 3 "" H 3900 4250 50  0001 C CNN
@@
 P 2600 4900
 F 0 "SW2" H 2700 5000 50  0000 C CNN
-F 1 "SW_Push" H 2600 4850 50  0000 C CNN
-F 2 "" H 2600 5100 50  0001 C CNN
+F 1 "RESET" H 2600 4850 50  0000 C CNN
+F 2 "thingy:SUNROM_4388" H 2600 5100 50  0001 C CNN
 F 3 "" H 2600 5100 50  0001 C CNN
 	1    2600 4900
@@
 P 4800 4300
 F 0 "J2" V 4750 4200 50  0000 L CNN
-F 1 "FLASH_JUMPER" V 4900 4350 50  0000 L CNN
+F 1 "FLASH" V 4900 4350 50  0000 L CNN
 F 2 "Connector_PinHeader_2.54mm:PinHeader_1x02_P2.54mm_Vertical" H 4800 4300 50  0001 C CNN
 F 3 "~" H 4800 4300 50  0001 C CNN
@@
 P 6850 5150
 F 0 "J3" H 7100 4850 50  0000 R CNN
-F 1 "Conn_01x04_Male" H 7400 5350 50  0000 R CNN
+F 1 "PROG" H 7400 5350 50  0000 R CNN
 F 2 "Connector_PinHeader_2.54mm:PinHeader_1x04_P2.54mm_Vertical" H 6850 5150 50  0001 C CNN
 F 3 "~" H 6850 5150 50  0001 C CNN
@@
 P 6850 5900
 F 0 "J4" H 7100 5600 50  0000 R CNN
-F 1 "Conn_01x04_Male" H 7400 6100 50  0000 R CNN
+F 1 "I2C" H 7400 6100 50  0000 R CNN
 F 2 "Connector_PinHeader_2.54mm:PinHeader_1x04_P2.54mm_Vertical" H 6850 5900 50  0001 C CNN
 F 3 "~" H 6850 5900 50  0001 C CNN
