File: pcb/thingy.kicad_pcb (KiCad board)
At the start: 2 copper layers, 1 part, among them U1 2x18650_holder

Commit message: few new elements & power module circuit
Parts:
- added J1: USB_B_Micro, Connector_USB:USB_Micro-B_Molex-105017-0001, F.Cu at (93.2, 99.3)
Connections:
- U1 pad 1: Net-(U1-Pad1) -> +5V
- U1 pad 3: Net-(U1-Pad3) -> GND
Routing:
- net GND: track 0.00 -> 245.6 mm, vias 0 -> 17

Commit message: more schematic work
Parts:
- added C1: 0.1u, Capacitor_SMD:C_1206_3216Metric, F.Cu at (142.7, 127.0)
- added C2: 10u, Capacitor_SMD:C_1206_3216Metric, F.Cu at (146.4, 122.0)
- added C3: 0.1u, Capacitor_SMD:C_1206_3216Metric, F.Cu at (134.5, 94.0)
- added D1: G, LED_SMD:LED_1206_3216Metric, F.Cu at (136.0, 109.2)
- added D2: R, LED_SMD:LED_1206_3216Metric, F.Cu at (135.1, 101.6)
- added J2: FLASH_JUMPER, Connector_PinHeader_2.54mm:PinHeader_1x02_P2.54mm_Vertical, F.Cu at (142.3, 119.2)
- added J3: Conn_01x04_Male, Connector_PinHeader_2.54mm:PinHeader_1x04_P2.54mm_Vertical, F.Cu at (119.9, 117.3)
- added R1: 100, Resistor_SMD:R_1206_3216Metric, F.Cu at (158.6, 107.3)
- added R10: 4k7, Resistor_SMD:R_1206_3216Metric, F.Cu at (151.0, 115.1)
- added R11: 4k7, Resistor_SMD:R_1206_3216Metric, F.Cu at (135.1, 79.2)
- added R12: 1k, Resistor_SMD:R_1206_3216Metric, F.Cu at (146.4, 115.1)
- added R2: 1k, Resistor_SMD:R_1206_3216Metric, F.Cu at (153.9, 109.7)
- added R3: 1k, Resistor_SMD:R_1206_3216Metric, F.Cu at (142.7, 124.7)
- added R4: 1k, Resistor_SMD:R_1206_3216Metric, F.Cu at (146.4, 119.7)
- added R5: 1k2, Resistor_SMD:R_1206_3216Metric, F.Cu at (135.0, 88.9)
- added R6: R, Resistor_SMD:R_1206_3216Metric, F.Cu at (135.0, 84.8)
- added R7: 4k7, Resistor_SMD:R_1206_3216Metric, F.Cu at (151.0, 112.7)
- added R8: 1k, Resistor_SMD:R_1206_3216Metric, F.Cu at (115.3, 100.1)
- added R9: 4k7, Resistor_SMD:R_1206_3216Metric, F.Cu at (146.4, 117.4)
- added U2: TP4056-B, Package_SO:SOIC-8_3.9x4.9mm_P1.27mm, F.Cu at (127.5, 106.2)
- added U3: 2x18650_holder, thingy:2x18650_holder, F.Cu at (120.3, 108.5)
- added U4: FS8205A, Package_SO:TSSOP-8_4.4x3mm_P0.65mm, F.Cu at (111.3, 118.9)
- added U5: ESP-07, RF_Module:ESP-07, F.Cu at (111.3, 85.3)
- U1: value 2x18650_holder -> DW01A; footprint thingy:2x18650_holder -> Package_TO_SOT_SMD:SOT-23-6
- moved J1 52.1 mm to (120.4, 143.8), turned to 0 degrees
- moved U1 32.1 mm to (115.8, 107.8)
Connections:
- U1 pad 1: +5V -> Net-(U1-Pad1)
- U1 pad 3: GND -> Net-(U1-Pad3)
Routing:
- net GND: track 245.6 -> 0.00 mm, vias 17 -> 0

Commit message: thingy work in progress
Parts:
- added J4: I2C, Connector_PinHeader_2.54mm:PinHeader_1x04_P2.54mm_Vertical, F.Cu at (154.6, 94.6)
- added SW1: POWER, thingy:MSS22D18, F.Cu at (122.7, 133.2)
- added SW2: RESET, thingy:SUNROM_4388, F.Cu at (106.8, 131.9)
- J2: value FLASH_JUMPER -> FLASH
- J3: value Conn_01x04_Male -> PROG
- moved C1 51.2 mm to (127.8, 78.0)
- moved C2 45.0 mm to (127.8, 81.0)
- moved R3 41.3 mm to (135.6, 84.0)
- moved R1 37.2 mm to (135.6, 78.0)
- moved U2 36.0 mm to (94.0, 119.3)
- moved R4 34.4 mm to (135.6, 87.0)
- moved R2 34.0 mm to (135.6, 81.0)
- moved R11 28.8 mm to (135.6, 108.0)
- moved R7 22.8 mm to (135.6, 96.0)
- moved D1 20.9 mm to (127.8, 90.0)
- moved R8 20.3 mm to (135.6, 99.0), turned to 180 degrees
- moved R9 18.8 mm to (135.6, 102.0)
- moved R10 18.4 mm to (135.6, 105.0)
- moved D2 16.3 mm to (127.8, 87.0)
- moved C3 12.0 mm to (127.8, 84.0)
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
Commit message: more work...
Parts:
- moved R2 56.2 mm to (120.0, 135.0)
- moved R5 53.5 mm to (103.9, 133.1), turned to 90 degrees
- moved R3 50.9 mm to (120.0, 132.4)
- moved D1 48.2 mm to (120.0, 137.6), turned to 180 degrees
- moved C3 47.7 mm to (110.8, 128.6), turned to 180 degrees
- moved R1 43.8 mm to (119.6, 118.8), turned to 270 degrees
- moved D2 43.5 mm to (120.0, 129.8), turned to 180 degrees
- moved C1 42.4 mm to (116.4, 118.8), turned to 90 degrees
- moved R6 39.0 mm to (106.4, 118.8), turned to 90 degrees
- moved R4 38.9 mm to (113.2, 118.8), turned to 270 degrees
- moved J4 35.9 mm to (124.5, 75.0), turned to 270 degrees
- moved R11 34.8 mm to (107.5, 87.4), turned to 270 degrees
- moved SW1 34.3 mm to (131.8, 100.1)
- moved R8 32.5 mm to (109.8, 118.8), turned to 270 degrees
- moved R10 31.1 mm to (110.0, 87.4), turned to 270 degrees
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Routing:
- net VCC: track 0.00 -> 48.9 mm, vias 0 -> 2
- net GND: track 0.00 -> 47.0 mm
- net I2C_SCL: track 0.00 -> 9.18 mm
- net I2C_SDA: track 0.00 -> 8.97 mm
- net Net-(J2-Pad2): track 0.00 -> 8.76 mm
- net Net-(R9-Pad2): track 0.00 -> 8.56 mm
- net Net-(R12-Pad1): track 0.00 -> 8.35 mm

Commit message: almost finished work on pcb
Parts:
- moved J4 9.19 mm to (116.0, 78.5), turned to 90 degrees
- moved U4 2.95 mm to (133.2, 122.2), turned to 0 degrees
- moved SW2 1.86 mm to (132.6, 133.6), turned to 180 degrees
- moved C3 1.09 mm to (110.8, 127.5)
- moved J1 0.90 mm to (120.3, 144.7)
- moved D2 0.77 mm to (120.0, 129.0)
- moved D1 0.58 mm to (120.0, 138.2)
- moved R5 0.57 mm to (103.6, 133.6), turned to 270 degrees
- moved R3 0.32 mm to (120.0, 132.1)
Routing:
- net BAT-: track 0.00 -> 69.4 mm, vias 0 -> 3
- net Net-(R6-Pad2): track 0.00 -> 54.6 mm, vias 0 -> 2
- net Net-(J2-Pad2): track 8.76 -> 58.3 mm
- net VCC: track 48.9 -> 0.00 mm, vias 2 -> 0
- net TXD: track 0.00 -> 37.6 mm, vias 0 -> 1
- net +5V: track 0.00 -> 35.1 mm
- net RXD: track 0.00 -> 33.9 mm, vias 0 -> 1
- net I2C_SCL: track 9.18 -> 33.1 mm
- net Net-(U1-Pad3): track 0.00 -> 22.0 mm, vias 0 -> 2
- net GND: track 47.0 -> 28.0 mm, vias 0 -> 11
- net I2C_SDA: track 8.97 -> 27.7 mm, vias 0 -> 1
- net Net-(SW1-Pad2): track 0.00 -> 16.4 mm
- net Net-(R4-Pad2): track 0.00 -> 16.0 mm
- net Net-(C1-Pad1): track 0.00 -> 15.9 mm, vias 0 -> 2
- net Net-(J1-Pad6): track 0.00 -> 12.0 mm
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- added copper zone on B.Cu, net GND
Other:
- board outline added: 40.4 x 77.8 mm
- net class POWER added: clearance 0.2, trace_width 0.3, via_dia 0.8, via_drill 0.4

Commit message: slightly more modifications
Routing:
- added copper zone on F.Cu, net VCC
Changed lines of the file:
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@@
+    )
+  )
+  (zone (net 9) (net_name VCC) (layer F.Cu) (hatch edge 0.508)
+    (connect_pads (clearance 0.508))
+    (min_thickness 0.254)
+    (fill yes (arc_segments 16) (thermal_gap 0.508) (thermal_bridge_width 0.508))
+    (polygon
+      (pts
+        (xy 100.08 69.6) (xy 100.08 147.44) (xy 140.43 147.44) (xy 140.43 69.6)
+      )
     )
   )
