File: pcb/thingy.kicad_pcb (KiCad board)
At the start: 2 copper layers, 40.4 x 77.8 mm, 28 parts, among them J1 USB_B_Micro, J2 FLASH, J3 PROG, J4 I2C, SW1 POWER, SW2 RESET, U1 DW01A, U2 TP4056-B, U3 2x18650_holder, U4 FS8205A, U5 ESP-07

Commit message: finished pcb v1.0
Parts:
- added REF**: OSHW-Logo2_7.3x6mm_SilkScreen, thingy:OSHW-Logo, F.Cu at (132.8, 78.6)
Other:
- board text added: "WTFPL LICENCE"
- board text added: "thingy ------ Paweł Tomaszewski"

Commit message: last fix
Parts:
- added REF**: BACK-IMG, thingy:BACK-IMG, F.Cu at (119.8, 109.0)
Other:
- board text added: "WTF Public Licence"
- board text added: "thingy v1.0 ------ Paweł Tomaszewski"
- board text removed: "WTFPL LICENCE"
- board text removed: "thingy ------ Paweł Tomaszewski"
Changed lines of the file:
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@@
     (tracks 213)
     (zones 0)
-    (modules 29)
+    (modules 30)
     (nets 35)
   )
@@
       (xy -2.549664 1.91989) (xy -2.469928 1.911165) (xy -2.400256 1.919918)) (layer F.SilkS) (width 0.01))
   )
-  (gr_text "WTFPL\nLICENCE" (at 105.66 77.72) (layer F.SilkS)
+  (module thingy:BACK-IMG (layer F.Cu)
+    (at 119.8 109)
+    (fp_text reference REF** (at -0.2 18.2) (layer F.SilkS)
+      (effects (font (size 1 1) (thickness 0.15)))
+    )
+    (fp_text value BACK-IMG (at 0 -11.9) (layer F.Fab)
+      (effects (font (size 1 1) (thickness 0.15)))
+    )
+    (fp_poly (pts (xy 6.8 -2.4) (xy 8.9 -1.7) (xy 5.6 0.1) (xy 3.3 -1)
+      (xy 3.7 -2.6) (xy 5.2 -1.3) (xy 6.8 -3.5) (xy 6.8 -2.7)) (layer B.SilkS) (width 0.15))
+    (fp_text user "NOT FOR IDIOTS" (at 0 3.9) (layer B.SilkS)
+      (effects (font (size 1 1) (thickness 0.15)) (justify mirror))
+    )
+    (fp_text user "SUPER DUPER PROJECT" (at 0.1 -3.8) (layer B.SilkS) hide
+      (effects (font (size 1 1) (thickness 0.15)) (justify mirror))
+    )
+    (fp_circle (center 0 0) (end 3 0) (layer B.SilkS) (width 0.15))
+    (fp_circle (center 0 0) (end 2.236068 0) (layer B.SilkS) (width 0.15))
+    (fp_circle (center 0 0) (end 1.414214 0) (layer B.SilkS) (width 0.15))
+  )
+  (gr_text "WTF\nPublic\nLicence" (at 105.4 75.7) (layer F.SilkS)
     (effects (font (size 1.5 1.5) (thickness 0.3)))
   )
-  (gr_text "thingy\n------\nPaweł\nTomaszewski" (at 127.29 89.2) (layer F.SilkS)
+  (gr_text "thingy v1.0\n------\nPaweł\nTomaszewski" (at 128.3 88.8) (layer F.SilkS)
     (effects (font (size 1.5 1.5) (thickness 0.3)))
   )
